Commit message: Firmware and controller.py upgrades for hand controller use

File: src/ipex_description/urdf/ipex.ros2_control.xacro (robot description, xacro)
@@ -1,4 +1,23 @@
 <?xml version="1.0"?>
 <robot xmlns:xacro="http://www.ros.org/wiki/xacro">
+  <!--
+    One <ros2_control> block per Teensy:
+      IPEXSystem      drivetrain Teensy (ipex_hardware/IpexSystem)
+      IPEXRearArm     rear arm Teensy   (ipex_hardware/IpexArmSystem)
+      IPEXFrontArm    front arm Teensy  (ipex_hardware/IpexArmSystem)
+    Arm blocks are enabled with xacro args rear_arm / front_arm.
+  -->
+  <xacro:arg name="rear_arm" default="true"/>
+  <xacro:arg name="front_arm" default="false"/>
+  <!-- Rear arm Teensy serial ID: set this. Find it with: ls /dev/serial/by-id/ -->
+  <xacro:arg name="rear_arm_serial_device"
+             default="/dev/serial/by-id/REAR_ARM_TEENSY_ID_NOT_SET"/>
+  <xacro:arg name="front_arm_serial_device"
+             default="/dev/serial/by-id/FRONT_ARM_TEENSY_ID_NOT_SET"/>
+  <!-- false: arms do NOT move on startup; home with /ipex/home_arms -->
+  <xacro:arg name="home_arms_on_start" default="false"/>
+  <!-- Must match firmware/arm/arm.ino MOTOR_STEPS_PER_REV -->
+  <xacro:property name="drum_steps_per_rev" value="400"/>
+  <!-- DRIVETRAIN -->
   <ros2_control name="IPEXSystem" type="system">
     <hardware>
@@ -15,31 +34,4 @@
       <param name="drivetrain_serial_baud">115200</param>
     </hardware>
-    <!-- SHOULDERS -->
-    <joint name="front_shoulder_rev">
-      <command_interface name="position"/>
-      <state_interface name="position"/>
-    </joint>
-    <joint name="back_shoulder_rev">
-      <command_interface name="position"/>
-      <state_interface name="position"/>
-    </joint>
-    <!-- DRUMS -->
-    <joint name="front_left_drum_rev">
-      <command_interface name="velocity"/>
-      <state_interface name="velocity"/>
-    </joint>
-    <joint name="front_right_drum_rev">
-      <command_interface name="velocity"/>
-      <state_interface name="velocity"/>
-    </joint>
-    <joint name="back_left_drum_rev">
-      <command_interface name="velocity"/>
-      <state_interface name="velocity"/>
-    </joint>
-    <joint name="back_right_drum_rev">
-      <command_interface name="velocity"/>
-      <state_interface name="velocity"/>
-    </joint>
-    <!-- DRIVETRAIN -->
     <joint name="front_left_wheel_rev">
       <command_interface name="velocity"/>
@@ -63,3 +55,36 @@
     </joint>
   </ros2_control>
+  <!-- ARMS: shoulder (position, rad) + two drums (velocity, rad/s, in sync) -->
+  <xacro:macro name="ipex_arm" params="block_name arm_name prefix device">
+    <ros2_control name="${block_name}" type="system">
+      <hardware>
+        <plugin>ipex_hardware/IpexArmSystem</plugin>
+        <param name="arm_name">${arm_name}</param>
+        <param name="serial_device">${device}</param>
+        <param name="serial_baud">115200</param>
+        <param name="drum_steps_per_rev">${drum_steps_per_rev}</param>
+        <param name="home_on_activate">$(arg home_arms_on_start)</param>
+      </hardware>
+      <joint name="${prefix}_shoulder_rev">
+        <command_interface name="position"/>
+        <state_interface name="position"/>
+      </joint>
+      <joint name="${prefix}_left_drum_rev">
+        <command_interface name="velocity"/>
+        <state_interface name="velocity"/>
+      </joint>
+      <joint name="${prefix}_right_drum_rev">
+        <command_interface name="velocity"/>
+        <state_interface name="velocity"/>
+      </joint>
+    </ros2_control>
+  </xacro:macro>
+  <xacro:if value="$(arg rear_arm)">
+    <xacro:ipex_arm block_name="IPEXRearArm" arm_name="rear_arm" prefix="back"
+                    device="$(arg rear_arm_serial_device)"/>
+  </xacro:if>
+  <xacro:if value="$(arg front_arm)">
+    <xacro:ipex_arm block_name="IPEXFrontArm" arm_name="front_arm" prefix="front"
+                    device="$(arg front_arm_serial_device)"/>
+  </xacro:if>
 </robot>

Commit message: Drum gear ratio added, drum speed in RPM on dpad

File: src/ipex_description/urdf/ipex.ros2_control.xacro (robot description, xacro)
@@ -19,6 +19,11 @@
   <!-- false: arms do NOT move on startup; home with /ipex/home_arms -->
   <xacro:arg name="home_arms_on_start" default="false"/>
-  <!-- Must match firmware/arm/arm.ino MOTOR_STEPS_PER_REV -->
-  <xacro:property name="drum_steps_per_rev" value="400"/>
+  <!-- Drum joint velocity is the DRUM (after the gearbox), so the hardware plugin
+       converts with motor steps per DRUM revolution:
+       firmware/arm/arm.ino MOTOR_STEPS_PER_REV (400) x drum gear ratio (80:1).
+       drum_gear_ratio must match teleop.yaml; primitives use the same 32000. -->
+  <xacro:property name="drum_motor_steps_per_rev" value="400"/>
+  <xacro:property name="drum_gear_ratio" value="80"/>
+  <xacro:property name="drum_steps_per_rev" value="${drum_motor_steps_per_rev * drum_gear_ratio}"/>
   <!-- DRIVETRAIN -->
   <ros2_control name="IPEXSystem" type="system">
